File: solar-0xFD02.sch (KiCad schematic (older format))
At the start: 25 parts, among them J1 Solar, J2 BAT, J3 ESP32, Q1 MOSFET, U1 CN3801

Commit message: Cleanup
Other:
- moved on the sheet: R3
Changed lines of the file:
@@
 L Device:R R3
 U 1 1 600DC61D
-P 1900 2000
-F 0 "R3" H 1970 2046 50  0000 L CNN
-F 1 "100k" H 1970 1955 50  0000 L CNN
-F 2 "Resistor_SMD:R_1206_3216Metric_Pad1.30x1.75mm_HandSolder" V 1830 2000 50  0001 C CNN
-F 3 "~" H 1900 2000 50  0001 C CNN
-	1    1900 2000
+P 1900 2250
+F 0 "R3" H 1970 2296 50  0000 L CNN
+F 1 "100k" H 1970 2205 50  0000 L CNN
+F 2 "Resistor_SMD:R_1206_3216Metric_Pad1.30x1.75mm_HandSolder" V 1830 2250 50  0001 C CNN
+F 3 "~" H 1900 2250 50  0001 C CNN
+	1    1900 2250
 	1    0    0    -1
 $EndComp
@@
 	3400 1250 3250 1250
 Wire Wire Line
-	1900 1850 1900 1250
+	1900 2100 1900 1250
 Connection ~ 1900 1250
 Wire Wire Line
@@
 	3600 2650 1900 2650
 Wire Wire Line
-	1900 2650 1900 2150
+	1900 2650 1900 2400
 $Comp
 L Device:R R4

Commit message: More cleanup
Parts:
- added C8: 100nF, Capacitor_SMD:C_1206_3216Metric_Pad1.33x1.80mm_HandSolder, symbol Device:CP1_Small
- added J4: BAT-, Connector_PinHeader_2.54mm:PinHeader_1x02_P2.54mm_Vertical, symbol Connector:Conn_01x02_Male
- added Q2: P-Chan, Package_TO_SOT_SMD:SOT-23, symbol Transistor_FET:AO3401A
- added U2: NCP302HSN30, Package_TO_SOT_SMD:SOT-23-5, symbol 0xFD:NCP302HSN30
- J3: renamed from J2; value BAT -> BAT+
- Q1: value MOSFET -> P-Chan
- renumbered J3 to J2
Connections:
- net labels added: Cd, ESP-LOAD, LVCO
- wire segments 93 -> 114
Other:
- moved on the sheet: C5, D2, D4, J2, J3, Q1, R6, R7, R8

Commit message: wip
Parts:
- added C9: 100nF, Capacitor_SMD:C_1206_3216Metric_Pad1.33x1.80mm_HandSolder, symbol Device:CP1_Small
Connections:
- wire segments 114 -> 120
Changed lines of the file:
@@
 	4850 6050 4850 6200
 Wire Wire Line
-	4850 6200 5100 6200
+	4850 6200 5000 6200
 Wire Wire Line
 	5400 6200 5850 6200
@@
 Connection ~ 5550 5300
 Wire Wire Line
-	5550 5300 4850 5300
+	5550 5300 5200 5300
 $Comp
 L Transistor_FET:AO3401A Q2
@@
 	1    0    0    -1
 $EndComp
+$Comp
+L Device:CP1_Small C9
+U 1 1 601C8E5A
+P 5200 5600
+F 0 "C9" V 4972 5600 50  0000 C CNN
+F 1 "100nF" V 5063 5600 50  0000 C CNN
+F 2 "Capacitor_SMD:C_1206_3216Metric_Pad1.33x1.80mm_HandSolder" H 5238 5450 50  0001 C CNN
+F 3 "~" H 5200 5600 50  0001 C CNN
+	1    5200 5600
+	-1   0    0    1
+$EndComp
+Wire Wire Line
+	5200 5500 5200 5300
+Connection ~ 5200 5300
+Wire Wire Line
+	5200 5300 4850 5300
+Wire Wire Line
+	5200 5700 5200 6050
+Wire Wire Line
+	5200 6050 5000 6050
+Wire Wire Line
+	5000 6050 5000 6200
+Connection ~ 5000 6200
+Wire Wire Line
+	5000 6200 5100 6200
 $EndSCHEMATC

Commit message: Added Zener diode and resistor for low voltage cutoff
Parts:
- added D5: D_Zener, Diode_SMD:D_1206_3216Metric_Pad1.42x1.75mm_HandSolder, symbol Device:D_Zener
- added R9: 10k, Resistor_SMD:R_1206_3216Metric_Pad1.30x1.75mm_HandSolder, symbol Device:R
Connections:
- wire segments 120 -> 126
Changed lines of the file:
@@
 	6650 2750 6650 2850
 Wire Wire Line
-	6200 4750 7300 4750
+	6200 4750 6350 4750
 Wire Wire Line
 	5850 4000 6900 4000
@@
 Text Label 6200 5550 0    50   ~ 0
 ESP-LOAD
-Text Label 6450 4750 0    50   ~ 0
+Text Label 7100 4750 0    50   ~ 0
 LVCO
 Text Label 5250 4600 0    50   ~ 0
@@
 Wire Wire Line
 	5000 6200 5100 6200
+$Comp
+L Device:D_Zener D5
+U 1 1 602F07BB
+P 6500 4750
+F 0 "D5" H 6500 4967 50  0000 C CNN
+F 1 "D_Zener" H 6500 4876 50  0000 C CNN
+F 2 "Diode_SMD:D_1206_3216Metric_Pad1.42x1.75mm_HandSolder" H 6500 4750 50  0001 C CNN
+F 3 "~" H 6500 4750 50  0001 C CNN
+	1    6500 4750
+	1    0    0    -1
+$EndComp
+Wire Wire Line
+	6650 4750 7000 4750
+$Comp
+L Device:R R9
+U 1 1 602F1515
+P 6550 3800
+F 0 "R9" V 6343 3800 50  0000 C CNN
+F 1 "10k" V 6434 3800 50  0000 C CNN
+F 2 "Resistor_SMD:R_1206_3216Metric_Pad1.30x1.75mm_HandSolder" V 6480 3800 50  0001 C CNN
+F 3 "~" H 6550 3800 50  0001 C CNN
+	1    6550 3800
+	0    1    1    0
+$EndComp
+Wire Wire Line
+	7000 4750 7000 3800
+Wire Wire Line
+	7000 3800 6700 3800
+Connection ~ 7000 4750
+Wire Wire Line
+	7000 4750 7300 4750
+Wire Wire Line
+	6400 3800 6150 3800
+Wire Wire Line
+	6150 3800 6150 3550
+Connection ~ 6150 3550
 $EndSCHEMATC

Commit message: Updated annotations
Parts:
- renumbered C6 to C1, C1 to C2, C7 to C3, C2 to C4, C3 to C5, C4 to C6, C8 to C7, C9 to C8, C5 to C9, D5 to D4, D4 to D5, J3 to J2, J4 to J3, J2 to J4, R5 to R1, R1 to R2, R2 to R5, R9 to R6, R6 to R8, R8 to R9
Other:
- moved on the sheet: C5, C6, R4, R5
Changed lines of the file:
@@
 NoConn ~ 3600 2550
 $Comp
-L Device:R R1
+L Device:R R2
 U 1 1 600DBBD4
 P 3050 1550
-F 0 "R1" H 3120 1596 50  0000 L CNN
+F 0 "R2" H 3120 1596 50  0000 L CNN
 F 1 "1k" H 3120 1505 50  0000 L CNN
 F 2 "Resistor_SMD:R_1206_3216Metric_Pad1.30x1.75mm_HandSolder" V 2980 1550 50  0001 C CNN
@@
 $EndComp
 $Comp
-L Device:CP1_Small C1
+L Device:CP1_Small C2
 U 1 1 600DCF7E
 P 2450 1550
-F 0 "C1" H 2541 1596 50  0000 L CNN
+F 0 "C2" H 2541 1596 50  0000 L CNN
 F 1 "10uF" H 2500 1450 50  0000 L CNN
 F 2 "Capacitor_SMD:C_1206_3216Metric_Pad1.33x1.80mm_HandSolder" H 2488 1400 50  0001 C CNN
@@
 $EndComp
 $Comp
-L Device:CP1_Small C2
+L Device:CP1_Small C4
 U 1 1 600DDAC2
 P 3800 1550
-F 0 "C2" H 3891 1596 50  0000 L CNN
+F 0 "C4" H 3891 1596 50  0000 L CNN
 F 1 "100nF" H 3891 1505 50  0000 L CNN
 F 2 "Capacitor_SMD:C_1206_3216Metric_Pad1.33x1.80mm_HandSolder" H 3838 1400 50  0001 C CNN
@@
 L Device:R R4
 U 1 1 600F7516
-P 1900 3000
-F 0 "R4" H 1970 3046 50  0000 L CNN
-F 1 "Rx" H 1970 2955 50  0000 L CNN
-F 2 "Resistor_SMD:R_1206_3216Metric_Pad1.30x1.75mm_HandSolder" V 1830 3000 50  0001 C CNN
-F 3 "~" H 1900 3000 50  0001 C CNN
-	1    1900 3000
-	1    0    0    -1
-$EndComp
-Wire Wire Line
-	1900 2650 1900 2850
+P 1900 2900
+F 0 "R4" H 1970 2946 50  0000 L CNN
+F 1 "Rx" H 1970 2855 50  0000 L CNN
+F 2 "Resistor_SMD:R_1206_3216Metric_Pad1.30x1.75mm_HandSolder" V 1830 2900 50  0001 C CNN
+F 3 "~" H 1900 2900 50  0001 C CNN
+	1    1900 2900
+	1    0    0    -1
+$EndComp
+Wire Wire Line
+	1900 2650 1900 2750
 Connection ~ 1900 2650
 Wire Wire Line
-	1900 3150 1900 3550
+	1900 3050 1900 3550
 Connection ~ 1900 3550
 Wire Wire Line
 	1900 3550 2100 3550
 $Comp
-L Device:R R2
+L Device:R R5
 U 1 1 600F8953
-P 4700 2900
-F 0 "R2" H 4770 2946 50  0000 L CNN
-F 1 "120" H 4770 2855 50  0000 L CNN
-F 2 "Resistor_SMD:R_1206_3216Metric_Pad1.30x1.75mm_HandSolder" V 4630 2900 50  0001 C CNN
-F 3 "~" H 4700 2900 50  0001 C CNN
-	1    4700 2900
-	1    0    0    -1
-$EndComp
-$Comp
-L Device:CP1_Small C4
+P 4700 3050
+F 0 "R5" H 4770 3096 50  0000 L CNN
+F 1 "120" H 4770 3005 50  0000 L CNN
+F 2 "Resistor_SMD:R_1206_3216Metric_Pad1.30x1.75mm_HandSolder" V 4630 3050 50  0001 C CNN
+F 3 "~" H 4700 3050 50  0001 C CNN
+	1    4700 3050
+	1    0    0    -1
+$EndComp
+$Comp
+L Device:CP1_Small C6
 U 1 1 600F9A74
-P 4700 3250
-F 0 "C4" H 4791 3296 50  0000 L CNN
-F 1 "220nF" H 4791 3205 50  0000 L CNN
-F 2 "Capacitor_SMD:C_1206_3216Metric_Pad1.33x1.80mm_HandSolder" H 4738 3100 50  0001 C CNN
-F 3 "~" H 4700 3250 50  0001 C CNN
-	1    4700 3250
+P 4700 3350
+F 0 "C6" H 4791 3396 50  0000 L CNN
+F 1 "220nF" H 4791 3305 50  0000 L CNN
+F 2 "Capacitor_SMD:C_1206_3216Metric_Pad1.33x1.80mm_HandSolder" H 4738 3200 50  0001 C CNN
+F 3 "~" H 4700 3350 50  0001 C CNN
+	1    4700 3350
 	1    0    0    -1
 $EndComp
@@
 	4400 2550 4700 2550
 Wire Wire Line
-	4700 2550 4700 2750
+	4700 2550 4700 2900
 Wire Wire Line
 	4700 3550 4250 3550
@@
 	5550 1250 5350 1250
 $Comp
-L Device:CP1_Small C3
+L Device:CP1_Small C5
 U 1 1 601047D3
-P 6150 1500
-F 0 "C3" H 6241 1546 50  0000 L CNN
-F 1 "22uF" H 6241 1455 50  0000 L CNN
-F 2 "Capacitor_SMD:C_1206_3216Metric_Pad1.33x1.80mm_HandSolder" H 6188 1350 50  0001 C CNN
-F 3 "~" H 6150 1500 50  0001 C CNN
-	1    6150 1500
+P 6150 2150
+F 0 "C5" H 6241 2196 50  0000 L CNN
+F 1 "22uF" H 6241 2105 50  0000 L CNN
+F 2 "Capacitor_SMD:C_1206_3216Metric_Pad1.33x1.80mm_HandSolder" H 6188 2000 50  0001 C CNN
+F 3 "~" H 6150 2150 50  0001 C CNN
+	1    6150 2150
 	1    0    0    -1
 $EndComp
@@
 Connection ~ 4950 3550
 $Comp
-L Connector:Conn_01x02_Male J3
+L Connector:Conn_01x02_Male J2
 U 1 1 60107AC2
 P 7000 2100
-F 0 "J3" H 7108 2281 50  0000 C CNN
+F 0 "J2" H 7108 2281 50  0000 C CNN
 F 1 "BAT+" H 7108 2190 50  0000 C CNN
 F 2 "Connector_PinHeader_2.54mm:PinHeader_1x02_P2.54mm_Vertical" H 7000 2100 50  0001 C CNN
@@
 	2450 1250 2450 1450
 Wire Wire Line
-	4700 3050 4700 3150
+	4700 3200 4700 3250
 Wire Wire Line
 	3800 1650 3800 1800
 Wire Wire Line
-	6150 1600 6150 2500
-Wire Wire Line
-	6150 1250 6150 1400
-Wire Wire Line
-	4700 3350 4700 3550
-$Comp
-L Device:R R5
+	6150 2250 6150 2500
+Wire Wire Line
+	6150 1250 6150 2050
+Wire Wire Line
+	4700 3450 4700 3550
+$Comp
+L Device:R R1
 U 1 1 60103D3F
 P 5850 1250
-F 0 "R5" V 5643 1250 50  0000 C CNN
+F 0 "R1" V 5643 1250 50  0000 C CNN
 F 1 "Rcs" V 5734 1250 50  0000 C CNN
 F 2 "Resistor_SMD:R_1206_3216Metric_Pad1.30x1.75mm_HandSolder" V 5780 1250 50  0001 C CNN
@@
 $EndComp
 $Comp
-L power:PWR_FLAG #FLG02
+L power:PWR_FLAG #FLG01
 U 1 1 6013116B
 P 3250 1250
-F 0 "#FLG02" H 3250 1325 50  0001 C CNN
+F 0 "#FLG01" H 3250 1325 50  0001 C CNN
 F 1 "PWR_FLAG" H 3250 1423 50  0000 C CNN
 F 2 "" H 3250 1250 50  0001 C CNN
@@
 	1650 3550 1900 3550
 $Comp
-L power:PWR_FLAG #FLG01
+L power:PWR_FLAG #FLG02
 U 1 1 60133894
 P 1650 2350
-F 0 "#FLG01" H 1650 2425 50  0001 C CNN
+F 0 "#FLG02" H 1650 2425 50  0001 C CNN
 F 1 "PWR_FLAG" V 1650 2477 50  0000 L CNN
 F 2 "" H 1650 2350 50  0001 C CNN
@@
 	4950 3550 5150 3550
 $Comp
-L Device:CP1_Small C5
+L Device:CP1_Small C9
 U 1 1 6024A6DF
 P 5700 5900
-F 0 "C5" V 5472 5900 50  0000 C CNN
+F 0 "C9" V 5472 5900 50  0000 C CNN
 F 1 "10uF" V 5563 5900 50  0000 C CNN
 F 2 "Capacitor_SMD:C_1206_3216Metric_Pad1.33x1.80mm_HandSolder" H 5738 5750 50  0001 C CNN
@@
 $EndComp
 $Comp
-L Device:LED D4
+L Device:LED D5
 U 1 1 6024B8B6
 P 4250 5750
-F 0 "D4" V 4197 5830 50  0000 L CNN
+F 0 "D5" V 4197 5830 50  0000 L CNN
 F 1 "LED" V 4288 5830 50  0000 L CNN
 F 2 "LED_SMD:LED_1206_3216Metric_Pad1.42x1.75mm_HandSolder" H 4250 5750 50  0001 C CNN
@@
 $EndComp
 $Comp
-L Device:R R8
+L Device:R R9
 U 1 1 6024C90E
 P 5250 6200
-F 0 "R8" V 5043 6200 50  0000 C CNN
+F 0 "R9" V 5043 6200 50  0000 C CNN
 F 1 "226k" V 5134 6200 50  0000 C CNN
 F 2 "Resistor_SMD:R_1206_3216Metric_Pad1.30x1.75mm_HandSolder" V 5180 6200 50  0001 C CNN
@@
 $EndComp
 $Comp
-L Connector:Conn_01x04_Female J2
+L Connector:Conn_01x04_Female J4
 U 1 1 6024DB17
 P 5750 6900
-F 0 "J2" V 5650 6550 50  0000 C CNN
+F 0 "J4" V 5650 6550 50  0000 C CNN
 F 1 "ESP32" V 5850 6850 50  0000 C CNN
 F 2 "Connector_PinHeader_2.54mm:PinHeader_1x04_P2.54mm_Vertical" H 5750 6900 50  0001 C CNN
@@
 $EndComp
 $Comp
-L Device:R R6
+L Device:R R8
 U 1 1 6024C2DF
 P 4250 6150
-F 0 "R6" H 4320 6196 50  0000 L CNN
+F 0 "R8" H 4320 6196 50  0000 L CNN
 F 1 "1k" H 4320 6105 50  0000 L CNN
 F 2 "Resistor_SMD:R_1206_3216Metric_Pad1.30x1.75mm_HandSolder" V 4180 6150 50  0001 C CNN
@@
 $EndComp
 $Comp
-L Device:CP1_Small C7
+L Device:CP1_Small C3
 U 1 1 602D4760
 P 2800 1550
-F 0 "C7" H 2900 1550 50  0000 L CNN
+F 0 "C3" H 2900 1550 50  0000 L CNN
 F 1 "100nF" H 2750 1450 50  0000 L CNN
 F 2 "Capacitor_SMD:C_1206_3216Metric_Pad1.33x1.80mm_HandSolder" H 2838 1400 50  0001 C CNN
@@
 	4850 3550 4850 5300
 $Comp
-L Device:CP1_Small C8
+L Device:CP1_Small C7
 U 1 1 601F4789
 P 5150 4200
-F 0 "C8" V 4922 4200 50  0000 C CNN
+F 0 "C7" V 4922 4200 50  0000 C CNN
 F 1 "100nF" V 5013 4200 50  0000 C CNN
 F 2 "Capacitor_SMD:C_1206_3216Metric_Pad1.33x1.80mm_HandSolder" H 5188 4050 50  0001 C CNN
@@
 	7300 5200 7200 5200
 $Comp
-L Connector:Conn_01x02_Male J4
+L Connector:Conn_01x02_Male J3
 U 1 1 6022E5F7
 P 7000 2850
-F 0 "J4" H 7108 3031 50  0000 C CNN
+F 0 "J3" H 7108 3031 50  0000 C CNN
 F 1 "BAT-" H 7108 2940 50  0000 C CNN
 F 2 "Connector_PinHeader_2.54mm:PinHeader_1x02_P2.54mm_Vertical" H 7000 2850 50  0001 C CNN
@@
 Cd
 $Comp
-L Device:CP1_Small C6
+L Device:CP1_Small C1
 U 1 1 602D4390
 P 2100 1550
-F 0 "C6" H 2191 1596 50  0000 L CNN
+F 0 "C1" H 2191 1596 50  0000 L CNN
 F 1 "10uF" H 2150 1450 50  0000 L CNN
 F 2 "Capacitor_SMD:C_1206_3216Metric_Pad1.33x1.80mm_HandSolder" H 2138 1400 50  0001 C CNN
@@
 $EndComp
 $Comp
-L Device:CP1_Small C9
+L Device:CP1_Small C8
 U 1 1 601C8E5A
 P 5200 5600
-F 0 "C9" V 4972 5600 50  0000 C CNN
+F 0 "C8" V 4972 5600 50  0000 C CNN
 F 1 "100nF" V 5063 5600 50  0000 C CNN
 F 2 "Capacitor_SMD:C_1206_3216Metric_Pad1.33x1.80mm_HandSolder" H 5238 5450 50  0001 C CNN
@@
 	5000 6200 5100 6200
 $Comp
-L Device:D_Zener D5
+L Device:D_Zener D4
 U 1 1 602F07BB
 P 6500 4750
-F 0 "D5" H 6500 4967 50  0000 C CNN
+F 0 "D4" H 6500 4967 50  0000 C CNN
 F 1 "D_Zener" H 6500 4876 50  0000 C CNN
 F 2 "Diode_SMD:D_1206_3216Metric_Pad1.42x1.75mm_HandSolder" H 6500 4750 50  0001 C CNN
@@
 	6650 4750 7000 4750
 $Comp
-L Device:R R9
+L Device:R R6
 U 1 1 602F1515
 P 6550 3800
-F 0 "R9" V 6343 3800 50  0000 C CNN
+F 0 "R6" V 6343 3800 50  0000 C CNN
 F 1 "10k" V 6434 3800 50  0000 C CNN
 F 2 "Resistor_SMD:R_1206_3216Metric_Pad1.30x1.75mm_HandSolder" V 6480 3800 50  0001 C CNN

Commit message: improvements and optimizations
Parts:
- added C5: 10uF, Capacitor_SMD:CP_Elec_3x5.4, symbol Device:CP1_Small
- added D4: LED, LED_SMD:LED_1206_3216Metric_Pad1.42x1.75mm_HandSolder, symbol Device:LED
- C1: footprint Capacitor_SMD:C_1206_3216Metric_Pad1.33x1.80mm_HandSolder -> Capacitor_SMD:CP_Elec_3x5.4
- C6: renamed from C5; value 22uF -> 10uF
- L1: footprint Inductor_SMD:L_1806_4516Metric_Pad1.57x1.80mm_HandSolder -> 0xFD:L-TYA4020
- U1: footprint solar-0xFD02:CN3801 -> 0xFD:CN3801
- renumbered C9 to C10, C6 to C7, C7 to C8, C8 to C9, D4 to D5, D5 to D6, R5 to R4, R4 to R5
Connections:
- net labels added: DONE
- wire segments 126 -> 135
- no-connect marks 1 -> 0
Other:
- note added: "Apache License\nVersion 2.0, January 2004\nhttp://www.apache.org/licenses/"
- moved on the sheet: C1, C10, C2, C3, C6, C7, C9, D1, D2, D3, D6, J1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

Commit message: Improvements
Parts:
- R1: value Rcs -> 0.24
- R3: value 100k -> 300k
- R5: value Rx -> 100k
Changed lines of the file:
@@
 P 1500 2150
 F 0 "R3" H 1570 2196 50  0000 L CNN
-F 1 "100k" H 1570 2105 50  0000 L CNN
+F 1 "300k" H 1570 2105 50  0000 L CNN
 F 2 "Resistor_SMD:R_1206_3216Metric_Pad1.30x1.75mm_HandSolder" V 1430 2150 50  0001 C CNN
 F 3 "~" H 1500 2150 50  0001 C CNN
@@
 P 1500 2950
 F 0 "R5" H 1570 2996 50  0000 L CNN
-F 1 "Rx" H 1570 2905 50  0000 L CNN
+F 1 "100k" H 1570 2905 50  0000 L CNN
 F 2 "Resistor_SMD:R_1206_3216Metric_Pad1.30x1.75mm_HandSolder" V 1430 2950 50  0001 C CNN
 F 3 "~" H 1500 2950 50  0001 C CNN
@@
 P 5850 1250
 F 0 "R1" V 5643 1250 50  0000 C CNN
-F 1 "Rcs" V 5734 1250 50  0000 C CNN
+F 1 "0.24" V 5734 1250 50  0000 C CNN
 F 2 "Resistor_SMD:R_1206_3216Metric_Pad1.30x1.75mm_HandSolder" V 5780 1250 50  0001 C CNN
 F 3 "~" H 5850 1250 50  0001 C CNN

Commit message: Made some footprints larger for easier soldering experience.
Parts:
- C1, C5: footprint Capacitor_SMD:CP_Elec_3x5.4 -> 0xFD:CP_Elec_3x6.4
- C10, C2, C3, C4, C6, C7, C8, C9: symbol Device:CP1_Small -> Device:C
- Q1: value P-Chan -> DMP1045U-7
- Q2: value P-Chan -> SSM3J332RLF
Connections:
- wire segments 135 -> 133
Changed lines of the file:
@@
 $EndComp
 $Comp
-L Device:CP1_Small C2
+L Device:C C2
 U 1 1 600DCF7E
-P 2200 1600
-F 0 "C2" H 2291 1646 50  0000 L CNN
-F 1 "10uF" H 2250 1500 50  0000 L CNN
-F 2 "Capacitor_SMD:C_1206_3216Metric_Pad1.33x1.80mm_HandSolder" H 2238 1450 50  0001 C CNN
-F 3 "~" H 2200 1600 50  0001 C CNN
-	1    2200 1600
-	1    0    0    -1
-$EndComp
-$Comp
-L Device:CP1_Small C4
+P 2200 1650
+F 0 "C2" H 2291 1696 50  0000 L CNN
+F 1 "10uF" H 2250 1550 50  0000 L CNN
+F 2 "Capacitor_SMD:C_1206_3216Metric_Pad1.33x1.80mm_HandSolder" H 2238 1500 50  0001 C CNN
+F 3 "~" H 2200 1650 50  0001 C CNN
+	1    2200 1650
+	1    0    0    -1
+$EndComp
+$Comp
+L Device:C C4
 U 1 1 600DDAC2
 P 3800 1550
@@
 $EndComp
 Wire Wire Line
-	3800 1250 3450 1250
-Wire Wire Line
 	3600 2150 3450 2150
 Connection ~ 3450 1250
@@
 Connection ~ 3050 1250
 Wire Wire Line
-	3050 1250 2550 1250
-Wire Wire Line
 	3050 1700 3050 1750
-Connection ~ 2200 1250
-Wire Wire Line
-	2200 1250 1850 1250
 Wire Wire Line
 	1000 1350 1200 1350
@@
 Wire Wire Line
 	4000 3550 4000 3000
-Wire Wire Line
-	2200 1700 2200 3550
-Connection ~ 2200 3550
 Wire Wire Line
 	1500 2650 1500 2300
@@
 $EndComp
 $Comp
-L Device:CP1_Small C7
+L Device:C C7
 U 1 1 600F9A74
-P 4650 3350
-F 0 "C7" H 4741 3396 50  0000 L CNN
-F 1 "220nF" H 4741 3305 50  0000 L CNN
-F 2 "Capacitor_SMD:C_1206_3216Metric_Pad1.33x1.80mm_HandSolder" H 4688 3200 50  0001 C CNN
-F 3 "~" H 4650 3350 50  0001 C CNN
-	1    4650 3350
+P 4650 3300
+F 0 "C7" H 4741 3346 50  0000 L CNN
+F 1 "220nF" H 4741 3255 50  0000 L CNN
+F 2 "Capacitor_SMD:C_1206_3216Metric_Pad1.33x1.80mm_HandSolder" H 4688 3150 50  0001 C CNN
+F 3 "~" H 4650 3300 50  0001 C CNN
+	1    4650 3300
 	1    0    0    -1
 $EndComp
@@
 	5550 1250 5450 1250
 $Comp
-L Device:CP1_Small C6
+L Device:C C6
 U 1 1 601047D3
 P 6150 2000
@@
 Connection ~ 6150 2500
 Wire Wire Line
-	3800 1250 3800 1450
-Wire Wire Line
-	2200 1250 2200 1500
-Wire Wire Line
-	4650 3000 4650 3250
-Wire Wire Line
-	3800 1650 3800 1800
-Wire Wire Line
-	6150 2100 6150 2250
-Wire Wire Line
 	6150 1250 6150 1700
 Wire Wire Line
@@
 Wire Wire Line
 	1200 2300 1200 3550
-Wire Wire Line
-	5050 3550 5150 3550
-$Comp
-L Device:CP1_Small C10
+$Comp
+L Device:C C10
 U 1 1 6024A6DF
 P 5700 6300
@@
 	5850 7200 5850 6300
 Wire Wire Line
-	5800 6300 5850 6300
-Wire Wire Line
-	5550 6300 5600 6300
-Wire Wire Line
 	5650 7200 5650 6850
 Wire Wire Line
@@
 Wire Wire Line
 	5750 7200 5750 6400
-Wire Wire Line
-	5750 6400 4750 6400
 Wire Wire Line
 	4250 6400 4250 6000
@@
 P 4100 1150
 F 0 "Q1" V 4000 1250 50  0000 C CNN
-F 1 "P-Chan" V 4350 1150 50  0000 C CNN
+F 1 "DMP1045U-7" V 4350 1150 50  0000 C CNN
 F 2 "Package_TO_SOT_SMD:SOT-23" H 4300 1075 50  0001 L CIN
 F 3 "https://www.mouser.com/datasheet/2/408/SSM3J332R_datasheet_en_20181015-1150575.pdf" V 4100 1150 50  0001 L CNN
@@
 $EndComp
 $Comp
-L Device:CP1_Small C3
+L Device:C C3
 U 1 1 602D4760
-P 2550 1600
-F 0 "C3" H 2650 1600 50  0000 L CNN
-F 1 "100nF" H 2500 1500 50  0000 L CNN
-F 2 "Capacitor_SMD:C_1206_3216Metric_Pad1.33x1.80mm_HandSolder" H 2588 1450 50  0001 C CNN
-F 3 "~" H 2550 1600 50  0001 C CNN
-	1    2550 1600
+P 2550 1650
+F 0 "C3" H 2650 1650 50  0000 L CNN
+F 1 "100nF" H 2500 1550 50  0000 L CNN
+F 2 "Capacitor_SMD:C_1206_3216Metric_Pad1.33x1.80mm_HandSolder" H 2588 1500 50  0001 C CNN
+F 3 "~" H 2550 1650 50  0001 C CNN
+	1    2550 1650
 	1    0    0    -1
 $EndComp
@@
 	1850 1700 1850 3550
 Connection ~ 1850 3550
-Wire Wire Line
-	1850 3550 2200 3550
-Wire Wire Line
-	2550 1250 2550 1500
-Connection ~ 2550 1250
-Wire Wire Line
-	2550 1250 2200 1250
 Text Label 4350 1250 0    50   ~ 0
 DRAIN
@@
 	4250 3550 4250 5300
 $Comp
-L Device:CP1_Small C8
+L Device:C C8
 U 1 1 601F4789
-P 5150 4200
-F 0 "C8" V 4922 4200 50  0000 C CNN
-F 1 "100nF" V 5013 4200 50  0000 C CNN
-F 2 "Capacitor_SMD:C_1206_3216Metric_Pad1.33x1.80mm_HandSolder" H 5188 4050 50  0001 C CNN
-F 3 "~" H 5150 4200 50  0001 C CNN
-	1    5150 4200
+P 5150 4150
+F 0 "C8" V 4922 4150 50  0000 C CNN
+F 1 "100nF" V 5013 4150 50  0000 C CNN
+F 2 "Capacitor_SMD:C_1206_3216Metric_Pad1.33x1.80mm_HandSolder" H 5188 4000 50  0001 C CNN
+F 3 "~" H 5150 4150 50  0001 C CNN
+	1    5150 4150
 	-1   0    0    1
 $EndComp
@@
 Wire Wire Line
 	5150 4600 5150 4300
-Wire Wire Line
-	5150 4100 5150 3550
-Connection ~ 5150 3550
-Wire Wire Line
-	5150 3550 6150 3550
 Wire Wire Line
 	5850 5150 5850 5300
@@
 Connection ~ 5550 6300
 Connection ~ 5550 5300
-Wire Wire Line
-	5550 5300 4750 5300
 $Comp
 L Transistor_FET:AO3401A Q2
@@
 P 7000 5200
 F 0 "Q2" H 6950 5050 50  0000 C CNN
-F 1 "P-Chan" V 7251 5200 50  0000 C CNN
+F 1 "SSM3J332RLF" V 7251 5200 50  0000 C CNN
 F 2 "Package_TO_SOT_SMD:SOT-23" H 7200 5125 50  0001 L CIN
 F 3 "https://www.mouser.com/datasheet/2/408/SSM3J332R_datasheet_en_20181015-1150575.pdf" V 7000 5200 50  0001 L CNN
@@
 Wire Wire Line
 	4300 1250 4600 1250
-Wire Wire Line
-	3800 1250 3900 1250
-Connection ~ 3800 1250
 Wire Wire Line
 	4100 1800 4100 1700
@@
 F 0 "C1" H 1941 1646 50  0000 L CNN
 F 1 "10uF" H 1900 1500 50  0000 L CNN
-F 2 "Capacitor_SMD:CP_Elec_3x5.4" H 1888 1450 50  0001 C CNN
+F 2 "0xFD:CP_Elec_3x6.4" H 1888 1450 50  0001 C CNN
 F 3 "~" H 1850 1600 50  0001 C CNN
 	1    1850 1600
@@
 $EndComp
 $Comp
-L Device:CP1_Small C9
+L Device:C C9
 U 1 1 601C8E5A
 P 4750 5600
@@
 	-1   0    0    1
 $EndComp
-Wire Wire Line
-	4750 5500 4750 5300
-Connection ~ 4750 5300
-Wire Wire Line
-	4750 5300 4250 5300
 $Comp
 L Device:D_Zener D5
@@
 F 0 "C5" H 5841 2046 50  0000 L CNN
 F 1 "10uF" H 5841 1955 50  0000 L CNN
-F 2 "Capacitor_SMD:CP_Elec_3x5.4" H 5788 1850 50  0001 C CNN
+F 2 "0xFD:CP_Elec_3x6.4" H 5788 1850 50  0001 C CNN
 F 3 "~" H 5750 2000 50  0001 C CNN
 	1    5750 2000
@@
 Wire Wire Line
 	5750 1700 6150 1700
-Connection ~ 6150 1700
-Wire Wire Line
-	6150 1700 6150 1900
 Wire Wire Line
 	5750 2100 5750 2250
 Wire Wire Line
 	5850 2400 6450 2400
-Connection ~ 6150 2250
 Wire Wire Line
 	6150 2250 6150 2500
@@
 	4250 3550 4000 3550
 Wire Wire Line
-	4250 6000 5050 6000
-Wire Wire Line
-	4750 5700 4750 6400
-Connection ~ 4750 6400
-Wire Wire Line
-	4750 6400 4250 6400
+	4250 6000 4750 6000
 Wire Wire Line
 	5750 2250 6150 2250
@@
 Wire Wire Line
 	3600 2650 1500 2650
-Wire Wire Line
-	2550 3550 3650 3550
-Connection ~ 2550 3550
-Wire Wire Line
-	2200 3550 2550 3550
-Wire Wire Line
-	2550 1700 2550 3550
 Text Label 3150 2650 0    50   ~ 0
 MPPT
 Text Notes 650  7600 0    79   ~ 0
 Apache License\nVersion 2.0, January 2004\nhttp://www.apache.org/licenses/
+Wire Wire Line
+	1850 1250 2200 1250
+Wire Wire Line
+	3450 1250 3800 1250
+Wire Wire Line
+	5050 3550 5150 3550
+Wire Wire Line
+	1850 3550 2200 3550
+Wire Wire Line
+	2200 1500 2200 1250
+Connection ~ 2200 1250
+Wire Wire Line
+	2200 1250 2550 1250
+Wire Wire Line
+	2550 1500 2550 1250
+Connection ~ 2550 1250
+Wire Wire Line
+	2550 1250 3050 1250
+Wire Wire Line
+	2200 1800 2200 3550
+Connection ~ 2200 3550
+Wire Wire Line
+	2200 3550 2550 3550
+Wire Wire Line
+	2550 1800 2550 3550
+Connection ~ 2550 3550
+Wire Wire Line
+	2550 3550 3650 3550
+Wire Wire Line
+	5150 4000 5150 3550
+Connection ~ 5150 3550
+Wire Wire Line
+	5150 3550 6150 3550
+Wire Wire Line
+	3800 1800 3800 1700
+Wire Wire Line
+	3800 1400 3800 1250
+Connection ~ 3800 1250
+Wire Wire Line
+	3800 1250 3900 1250
+Wire Wire Line
+	6150 2150 6150 2250
+Connection ~ 6150 2250
+Wire Wire Line
+	6150 1850 6150 1700
+Connection ~ 6150 1700
+Wire Wire Line
+	4650 3150 4650 3000
+Wire Wire Line
+	4250 6400 5750 6400
+Wire Wire Line
+	4750 5450 4750 5300
+Wire Wire Line
+	4250 5300 4750 5300
+Connection ~ 4750 5300
+Wire Wire Line
+	4750 5300 5550 5300
+Wire Wire Line
+	4750 5750 4750 6000
+Connection ~ 4750 6000
+Wire Wire Line
+	4750 6000 5050 6000
 $EndSCHEMATC
