File: solar-0xFD02.sch (KiCad schematic (older format))
At the start: 34 parts, among them J1 Solar, J2 BAT+, J3 BAT-, J4 ESP32, Q1 DMP1045U-7, Q2 SSM3J332RLF, U1 CN3801, U2 NCP302HSN30

Commit message: Fixed zener diode pad
Parts:
- D5: footprint Diode_SMD:D_1206_3216Metric_Pad1.42x1.75mm_HandSolder -> Diode_SMD:D_SOD-123
Changed lines of the file:
@@
 	5850 6000 5850 6300
 Wire Wire Line
-	5750 7200 5750 6400
-Wire Wire Line
-	4250 6400 4250 6000
+	5750 7200 5750 6500
+Wire Wire Line
+	4250 6500 4250 6000
 Connection ~ 4250 6000
 Text Label 3150 3550 0    50   ~ 0
@@
 Text Label 2050 1250 0    50   ~ 0
 SOL+
-Text Label 5150 6400 0    50   ~ 0
+Text Label 5150 6500 0    50   ~ 0
 ADC
 Text Label 4350 6850 0    50   ~ 0
@@
 F 0 "D5" H 6500 4967 50  0000 C CNN
 F 1 "D_Zener" H 6500 4876 50  0000 C CNN
-F 2 "Diode_SMD:D_1206_3216Metric_Pad1.42x1.75mm_HandSolder" H 6500 4750 50  0001 C CNN
+F 2 "Diode_SMD:D_SOD-123" H 6500 4750 50  0001 C CNN
 F 3 "~" H 6500 4750 50  0001 C CNN
 	1    6500 4750
@@
 	4650 3150 4650 3000
 Wire Wire Line
-	4250 6400 5750 6400
+	4250 6500 5750 6500
 Wire Wire Line
 	4750 5450 4750 5300
